Commit message: feat: wire launch master_id into Ethercat master construction

File: brainco_hardware/stark_ethercat/brainco_hand_ethercat_driver/config/revo2_left.ros2_control.xacro (robot description, xacro)
@@ -1,5 +1,5 @@
 <?xml version="1.0"?>
 <robot xmlns:xacro="http://www.ros.org/wiki/xacro">
-    <xacro:macro name="revo2_left_ros2_control" params="name initial_positions_file ctrl_param_duration_ms:=10">
+    <xacro:macro name="revo2_left_ros2_control" params="name initial_positions_file ctrl_param_duration_ms:=10 master_id:=0">
         <xacro:property name="initial_positions" value="${xacro.load_yaml(initial_positions_file)['initial_positions']}"/>
         <ros2_control name="${name}" type="system">
@@ -7,5 +7,5 @@
                 <!-- Use EtherCAT driver for real hardware -->
                 <plugin>stark_ethercat_driver/EthercatDriver</plugin>
-                <param name="master_id">0</param>
+                <param name="master_id">${master_id}</param>
                 <param name="control_frequency">1000</param>
             </hardware>

File: brainco_hardware/stark_ethercat/brainco_hand_ethercat_driver/config/revo2_left.urdf.xacro (robot description, xacro)
@@ -3,4 +3,5 @@
     <xacro:arg name="initial_positions_file" default="revo2_left_initial_positions.yaml" />
     <xacro:arg name="ctrl_param_duration_ms" default="10" />
+    <xacro:arg name="master_id" default="0" />
     <!-- World link -->
     <link name="world"/>
@@ -16,4 +17,4 @@
     <!-- Import ros2_control configuration -->
     <xacro:include filename="revo2_left.ros2_control.xacro" />
-    <xacro:revo2_left_ros2_control name="Revo2LeftEthercatSystem" initial_positions_file="$(arg initial_positions_file)" ctrl_param_duration_ms="$(arg ctrl_param_duration_ms)"/>
+    <xacro:revo2_left_ros2_control name="Revo2LeftEthercatSystem" initial_positions_file="$(arg initial_positions_file)" ctrl_param_duration_ms="$(arg ctrl_param_duration_ms)" master_id="$(arg master_id)"/>
 </robot>

File: brainco_hardware/stark_ethercat/brainco_hand_ethercat_driver/config/revo2_right.ros2_control.xacro (robot description, xacro)
@@ -1,5 +1,5 @@
 <?xml version="1.0"?>
 <robot xmlns:xacro="http://www.ros.org/wiki/xacro">
-    <xacro:macro name="revo2_right_ros2_control" params="name initial_positions_file ctrl_param_duration_ms:=10">
+    <xacro:macro name="revo2_right_ros2_control" params="name initial_positions_file ctrl_param_duration_ms:=10 master_id:=0">
         <xacro:property name="initial_positions" value="${xacro.load_yaml(initial_positions_file)['initial_positions']}"/>
         <ros2_control name="${name}" type="system">
@@ -7,5 +7,5 @@
                 <!-- Use EtherCAT driver for real hardware -->
                 <plugin>stark_ethercat_driver/EthercatDriver</plugin>
-                <param name="master_id">0</param>
+                <param name="master_id">${master_id}</param>
                 <param name="control_frequency">1000</param>
             </hardware>

File: brainco_hardware/stark_ethercat/brainco_hand_ethercat_driver/config/revo2_right.urdf.xacro (robot description, xacro)
@@ -3,4 +3,5 @@
     <xacro:arg name="initial_positions_file" default="revo2_right_initial_positions.yaml" />
     <xacro:arg name="ctrl_param_duration_ms" default="10" />
+    <xacro:arg name="master_id" default="0" />
     <!-- World link -->
     <link name="world"/>
@@ -16,4 +17,4 @@
     <!-- Import ros2_control configuration -->
     <xacro:include filename="revo2_right.ros2_control.xacro" />
-    <xacro:revo2_right_ros2_control name="Revo2RightEthercatSystem" initial_positions_file="$(arg initial_positions_file)" ctrl_param_duration_ms="$(arg ctrl_param_duration_ms)"/>
+    <xacro:revo2_right_ros2_control name="Revo2RightEthercatSystem" initial_positions_file="$(arg initial_positions_file)" ctrl_param_duration_ms="$(arg ctrl_param_duration_ms)" master_id="$(arg master_id)"/>
 </robot>
